File: kicad/small/power_injector_rev_c.kicad_pcb (KiCad board)
At the start: 2 copper layers, 72 x 20 mm, 15 parts, among them J2 A00-108-220-450, J3 A00-108-220-450

Commit message: Added screw terminal version
Other:
- board text added: "24V"
